Commit message: Corregido algunos fallos y driver detectado ya

File: super_lane_pkg/resource/CitroenCZero.urdf (robot description, URDF)
Before this commit: robot /home/hugo/Documentos/RO/Practica1-RO/super_lane_pkg/resource/CitroenCZero.urdf, 13 links, 14 joints
Links:
- removed link antifog_lights
- removed link backwards_lights
- removed link base_link
- removed link brake_lights
- removed link car_camera
- removed link engine_speaker
- removed link front_lights
- removed link left_indicators
- removed link rear left wheel
- removed link rear right wheel
- removed link rear_lights
- removed link right_indicators
- removed link road_camera
Joints:
- removed joint base_link_antifog_lights_joint
- removed joint base_link_backwards_lights_joint
- removed joint base_link_brake_lights_joint
- removed joint base_link_car_camera_joint
- removed joint base_link_engine_speaker_joint
- removed joint base_link_front_lights_joint
- removed joint base_link_left_indicators_joint
- removed joint base_link_rear_lights_joint
- removed joint base_link_right_indicators_joint
- removed joint base_link_road_camera_joint
- removed joint left_rear_wheel
- removed joint right_rear_wheel
- removed joint slot_0_rear left wheel_joint
- removed joint slot_rear right wheel_joint
